Commit message: Now it is working on gazebo

File: robot/single_lwr_robot.urdf.xacro (robot description, xacro)
@@ -5,4 +5,9 @@
 	<xacro:include filename="$(find end_effector)/urdf/end_effector.urdf.xacro" />
 	<!-- and assemble your robot -->
+	<link name="world"/>
+	<joint name="fixed_w" type="fixed">
+      <parent link="world"/>
+      <child link="box"/>
+    </joint>
 	<link name="box">
 		<inertial>
@@ -27,13 +32,13 @@
 		</collision>
 	</link>
-	<gazebo reference="box">
-		<static>true</static>>
-	</gazebo>
+<!-- 	<gazebo reference="box">
+		<static>true</static>
+	</gazebo -->>
 	<!-- using the models -->
 	<xacro:kuka_lwr parent="box" name="lwr">
 		<origin xyz="0 0 1" rpy="0 0 0"/>
 	</xacro:kuka_lwr>
-	<xacro:end_effector_kuka_lwr parent="lwr_7_link" name="lwr_end_effector">
-		<origin xyz="0 0 1" rpy="0 0 0"/>
+	<xacro:end_effector_kuka_lwr parent="lwr_7_link" name="lwr">
+		<origin xyz="0 0 0" rpy="0 0 0"/>
 	</xacro:end_effector_kuka_lwr>
 </robot>

File: urdf/end_effector.urdf.xacro (robot description, xacro)
@@ -1,142 +1,83 @@
 <?xml version="1.0"?>
-<!-- Revolute-Revolute Manipulator -->
-<robot name="end_effector" xmlns:xacro="http://www.ros.org/wiki/xacro">
+<robot xmlns:xacro="http://www.ros.org/wiki/xacro" name="end_effector">
   <!-- Constants for robot dimensions -->
   <xacro:property name="PI" value="3.1415926535897931"/>
-  <xacro:property name="mass" value="1" /> <!-- arbitrary value for mass -->
+  <xacro:property name="mass" value="0.001" /> <!-- arbitrary value for mass -->
   <xacro:property name="width" value="0.25" />
   <xacro:property name="height" value="0.5" />
-  <xacro:property name="length" value="0.25" />
-  <xacro:property name="radius" value="0.125" /> <!-- Square dimensions (widthxwidth) of beams -->
+  <xacro:property name="length" value="0.025" />
+  <xacro:property name="radius" value="0.05" />
   <!-- Import all Gazebo-customization elements, including Gazebo colors -->
   <xacro:include filename="$(find end_effector)/urdf/end_effector.gazebo" />
-  <!-- Import Rviz colors -->
-  <!-- <xacro:include filename="$(find rrbot_description)/urdf/materials.xacro" /> -->
-  <!--xacro:include filename="$(find lwr_description)/model/kuka_lwr.gazebo.xacro"/-->
   <xacro:macro name="end_effector_kuka_lwr" params="parent name *origin">
-  <!-- Used for fixing robot to Gazebo 'base_link' -->
-  <!-- <link name="world"/> -->
-  <joint name="fixed" type="fixed">
-    <parent link="${parent}"/>
-    <child link="link_cubo1"/>
-  </joint>
-  <!-- Base Link -->
-  <link name="link_cubo1">
-    <collision>
-      <origin xyz="0 0 ${height/2}" rpy="0 0 0"/>
+    <joint name="fixed" type="fixed">
+      <parent link="${parent}"/>
+      <child link="link_cubo1"/>
+      <xacro:insert_block name="origin"/>
+    </joint>
+    <link name="link_cubo1">
+      <collision>
+      <origin xyz="0 0 0" rpy="0 0 0"/>
       <geometry>
-	<box size="${length} ${width} ${height}"/>
+        <cylinder radius="${radius}" length="${length}"/>
       </geometry>
-    </collision>
-    <visual>
-      <origin xyz="0 0 ${height/2}" rpy="0 0 0"/>
-      <geometry>
-	<box size="${length} ${width} ${height}"/>
-      </geometry>
-      <material name="orange"/>
-    </visual>
-    <inertial>
-      <origin xyz="0 0 ${height/2}" rpy="0 0 0"/>
-      <mass value="${mass}"/>
-      <inertia
-	  ixx="${mass / 12.0 * (height*height + length*length)}" ixy="0.0" ixz="0.0"
-	  iyy="${mass / 12.0 * (width*width + length*length)}" iyz="0.0"
-	  izz="${mass / 12.0 * (width*width + height*height)}"/>
-    </inertial>
-  </link>
-  <joint name="joint1" type="revolute">
-    <parent link="link_cubo1"/>
-    <child link="link_cubo2"/>
-    <origin xyz="0 0 ${width}" rpy="0 0 0"/>
-    <axis xyz="0 0 1"/>
-    <limit lower="0" upper="0" effort="0" velocity="0"/>
-    <!-- <dynamics damping="0.7"/> -->
-  </joint>
-  <!-- Middle Link -->
-  <link name="link_cubo2">
-    <collision>
-      <origin xyz="0 0 ${0.75*height}" rpy="0 0 0"/>
-      <geometry>
-	<box size="${height} ${width} ${length}"/>
-      </geometry>
-    </collision>
-    <visual>
-      <origin xyz="0 0 ${0.75*height}" rpy="0 0 0"/>
-      <geometry>
-	<box size="${height} ${width} ${length}"/>
-      </geometry>
-      <material name="black"/>
-    </visual>
-    <inertial>
-      <origin xyz="${height/2} ${width/2} ${length/2}" rpy="0 0 0"/>
-      <mass value="${mass}"/>
-      <inertia
-    ixx="${mass / 12.0 * (length*length + height*height)}" ixy="0.0" ixz="0.0"
-    iyy="${mass / 12.0 * (width*width + height*height)}" iyz="0.0"
-    izz="${mass / 12.0 * (width*width + length*length)}"/>
-    </inertial>
-  </link>
-  <joint name="fixed1" type="fixed">
-    <parent link="link_cubo2"/>
-    <child link="link_cubo3"/>
-  </joint>
-  <link name="link_cubo3">
-    <collision>
-      <origin xyz="0 0 ${1.5*height}" rpy="0 0 0"/>
-      <geometry>
-  <box size="${length} ${width} ${height}"/>
-      </geometry>
-    </collision>
-    <visual>
-      <origin xyz="0 0 ${height*1.5}" rpy="0 0 0"/>
-      <geometry>
-  <box size="${length} ${width} ${height}"/>
-      </geometry>
-    </visual>
-    <inertial>
-      <origin xyz="${length/2} ${width/2} ${height/2}" rpy="0 0 0"/>
-      <mass value="${mass}"/>
-      <inertia
-    ixx="${mass / 12.0 * (height*height + length*length)}" ixy="0.0" ixz="0.0"
-    iyy="${mass / 12.0 * (width*width + length*length)}" iyz="0.0"
-    izz="${mass / 12.0 * (width*width + height*height)}"/>
-    </inertial>
-  </link>
-  <joint name="fixed2" type="fixed">
-    <parent link="link_cubo3"/>
-    <child link="link_sfera"/>
-  </joint>
-<link name="link_sfera">
-    <collision>
-      <origin xyz="0 0 0.375" rpy="0 0 0"/>
-      <geometry>
-  <sphere radius="${radius}"/>
-      </geometry>
-    </collision>
-    <visual>
-      <origin xyz="0 0 1" rpy="0 0 0"/>
-      <geometry>
-  <sphere radius="${radius}"/>
-      </geometry>
-    </visual>
-    <!--inertial>
-      <origin xyz="0 0 ${height/2}" rpy="0 0 0"/>
-      <mass value="${mass}"/>
-      <inertia
-    ixx="${mass / 12.0 * (height*height + length*length)}" ixy="0.0" ixz="0.0"
-    iyy="${mass / 12.0 * (width*width + length*length)}" iyz="0.0"
-    izz="${mass / 12.0 * (width*width + height*height)}"/>
-    </inertial-->
-  </link>
-  <transmission name="tran1">
-    <type>transmission_interface/SimpleTransmission</type>
-    <joint name="joint1">
-      <hardwareInterface>EffortJointInterface</hardwareInterface>
+      </collision>
+      <visual>
+        <origin xyz="0 0 0" rpy="0 0 0"/>
+        <geometry>
+          <cylinder radius="${radius}" length="${length}"/>
+        </geometry>
+        <material name="orange"/>
+      </visual>
+      <inertial>
+        <mass value="${mass}"/>
+        <origin xyz="0 0 0"  />
+        <cylinder_inertia_def radius="0.05" length="0.025" mass="${mass}"/>
+      </inertial>
+    </link>
+    <joint name="joint1" type="fixed">
+      <parent link="link_cubo1"/>
+      <child link="link_cubo2"/>
+      <origin xyz="0 0 0.025" rpy="0 0 0"/>
     </joint>
-    <actuator name="motor1">
-      <hardwareInterface>EffortJointInterface</hardwareInterface>
-      <mechanicalReduction>1</mechanicalReduction>
-    </actuator>
-  </transmission>
-    </xacro:macro>
+    <link name="link_cubo2">
+      <collision>
+        <origin xyz="0 0 0" rpy="0 0 0"/>
+        <geometry>
+          <cylinder radius="${radius}" length="${length}"/>
+        </geometry>
+      </collision>
+      <visual>
+        <origin xyz="0 0 0" rpy="0 0 0"/>
+        <geometry>
+          <cylinder radius="${radius}" length="${length}"/>
+        </geometry>
+        <material name="orange"/>
+      </visual>
+      <inertial>
+        <mass value="${mass}"/>
+        <origin xyz="0 0 0"  />
+        <cylinder_inertia_def radius="0.05" length="0.025" mass="${mass}"/>
+      </inertial>
+    </link>
+    <joint name="fixed2" type="fixed">
+      <parent link="link_cubo2"/>
+      <child link="link_sfera"/>
+    </joint>
+    <link name="link_sfera">
+      <collision>
+        <origin xyz="0 0 0.005" rpy="0 0 0"/>
+        <geometry>
+          <sphere radius="${radius}"/>
+        </geometry>
+      </collision>
+      <visual>
+        <origin xyz="0 0 0.005" rpy="0 0 0"/>
+        <geometry>
+          <sphere radius="${radius}"/>
+        </geometry>
+      </visual>
+    </link>
+  </xacro:macro>
+  <xacro:kuka_lwr_gazebo_ft_sensor name="lwr"/>
 </robot>

Commit message: testing force sensor

File: robot/single_lwr_robot.urdf.xacro (robot description, xacro)
@@ -42,3 +42,18 @@
 		<origin xyz="0 0 0" rpy="0 0 0"/>
 	</xacro:end_effector_kuka_lwr>
+	<joint name="fixed_ef" type="fixed">
+		<origin xyz="0 0 0.0875" rpy="0 0 0"/>
+      <parent link="lwr_7_link"/>
+      <child link="ef"/>
+    </joint>
+	<link name="ef">
+		<inertial>
+			<mass value="0.001"/>
+			<origin rpy="0 0 0" xyz="0 0 0"/>
+			<inertia ixx="0.001"
+             iyy="0.001"
+             izz="0.001"
+             ixy="0" iyz="0" ixz="0"/>
+		</inertial>
+	</link>
 </robot>

File: urdf/box.urdf.xacro (robot description, xacro)
@@ -1,14 +1,15 @@
 <?xml version="1.0"?>
 <robot xmlns:xacro="http://www.ros.org/wiki/xacro" name="box">
+<link name="world"/>
 <link name="box">
    <inertial>
-       <origin xyz="-1 0 0" rpy="0 0 0" />
+       <origin xyz="-0.6 0 0" rpy="0 0 0" />
      <mass value="1000"/>
      <inertia ixx="1666.6667"  ixy="0"  ixz="0" iyy="1666.6667" iyz="0" izz="2666.6667" />
    </inertial>
    <visual>
-     <origin xyz="-1 0 0" rpy="0 0 0" />
+     <origin xyz="-0.6 0 0" rpy="0 0 0" />
      <geometry>
-       <box size="2 4 4" />
+       <box size="1 2 2" />
      </geometry>
   <material name="Kuka/Red">
@@ -17,17 +18,16 @@
    </visual>
    <collision>
-   	<origin xyz="-1 0 0" rpy="0 0 0" />
+   	<origin xyz="-0.6 0 0" rpy="0 0 0" />
      <geometry>
-     <box size="2 4 4" />
+     <box size="1 2 2" />
      </geometry>
    </collision>
  </link>
-	<!-- <gazebo reference="cylinder"> -->
-		<!--selfCollide>true</selfCollide-->
-		<!-- <gravity>false</gravity> -->
-		<!-- <mu1>1.0</mu1> -->
-		<!-- <mu2>1.0</mu2> -->
-		<!-- <kp>10000000.0</kp> -->
-		<!-- <kd>1.0</kd> -->
-	<!-- </gazebo> -->
+<joint name="prismatic_joint" type="fixed">
+    <parent link="world"/>
+    <child link="box"/>
+    <!-- <limit effort="1000.0" lower="-0.01" upper="0.01" velocity="0.001"/> -->
+    <origin xyz="0 0 0" rpy="0 0 0" />
+    <!-- <axis xyz="0 1 0"/> -->
+  </joint>
 </robot>
